Commit message: slam

File: urdf/myrobot.urdf (robot description, URDF)
Before this commit: robot my_robot, 7 links, 6 joints
Links:
- removed link depth_camera
- removed link lidar
- added link depth_camera_link; visual box size=0.05 0.05 0.05
- added link imu_link
- added link lidar_link; visual cylinder length=0.05 radius=0.05
Joints:
- added joint imu_joint: type fixed, parent base_link, child imu_link, origin xyz=0 0 0.15
- joint depth_camera_joint: child depth_camera -> depth_camera_link; origin xyz=0.30 0 0.25 -> xyz=0.30 0 0.20
- joint lidar_joint: child lidar -> lidar_link
