Commit message: Complete ROS-Gazebo pipeline: 4-wheel URDF with GPS+depth-cam, vertical ArUco boards, EKF local+global, SLAM mapping/localization mode, Nav2 waypoint + ArUco chain missions

File: urdf/myrobot.urdf (robot description, URDF)
Before this commit: robot my_robot, 8 links, 7 joints
Links:
- removed link caster_wheel
- removed link left_wheel
- removed link right_wheel
- added link front_left_wheel, mass 0.8; collision cylinder length=0.05 radius=0.1; visual cylinder length=0.05 radius=0.1
- added link front_right_wheel, mass 0.8; collision cylinder length=0.05 radius=0.1; visual cylinder length=0.05 radius=0.1
- added link gps_link, mass 0.1; collision box size=0.06 0.06 0.03; visual box size=0.06 0.06 0.03
- added link rear_left_wheel, mass 1.0; collision cylinder length=0.05 radius=0.1; visual cylinder length=0.05 radius=0.1
- added link rear_right_wheel, mass 1.0; collision cylinder length=0.05 radius=0.1; visual cylinder length=0.05 radius=0.1
- link depth_camera_link: mass None -> 0.2; geometry collision box size=0.05 0.05 0.05; visual box size=0.05 0.05 0.05
- link imu_link: mass None -> 0.1
- link lidar_link: mass None -> 0.3; geometry collision cylinder length=0.05 radius=0.05; visual cylinder length=0.05 radius=0.05
Joints:
- removed joint caster_joint
- removed joint left_wheel_joint
- removed joint right_wheel_joint
- added joint front_left_wheel_joint: type continuous, parent base_link, child front_left_wheel, origin xyz=0.20 0.20 0.10 rpy=0 0 0, axis 0 1 0
- added joint front_right_wheel_joint: type continuous, parent base_link, child front_right_wheel, origin xyz=0.20 -0.20 0.10 rpy=0 0 0, axis 0 1 0
- added joint gps_joint: type fixed, parent base_link, child gps_link, origin xyz=-0.10 0 0.22 rpy=0 0 0
- added joint rear_left_wheel_joint: type continuous, parent base_link, child rear_left_wheel, origin xyz=-0.15 0.20 0.10 rpy=0 0 0, axis 0 1 0
- added joint rear_right_wheel_joint: type continuous, parent base_link, child rear_right_wheel, origin xyz=-0.15 -0.20 0.10 rpy=0 0 0, axis 0 1 0
- joint base_joint: origin (none) -> xyz=0 0 0 rpy=0 0 0
- joint depth_camera_joint: origin xyz=0.30 0 0.20 -> xyz=0.30 0 0.20 rpy=0 0 0
- joint imu_joint: origin xyz=0 0 0.15 -> xyz=0 0 0.15 rpy=0 0 0
- joint lidar_joint: origin xyz=0 0 0.25 -> xyz=0 0 0.25 rpy=0 0 0
